File: drone_controller.kicad_pcb (KiCad board)
At the start: 2 copper layers, 40.3 x 16.2 mm, 18 parts, among them J1 Conn_01x03_Pin, P1 PAD, P2 PAD, P3 PAD, P4 PAD, Q1 AGM60P100A, Q2 BSS138LT3G, SW1 SW_SPDT, U1 2060-452/998-404, U2 2060-452/998-404

Commit message: v2.0 release production freeze
Parts:
- removed C1: C_Polarized, easyeda2kicad:CAP-TH_BD8.0-P3.50-D0.6-FD
- removed D1: LED_R, easyeda2kicad:LED0402-RD
- removed D2: LED_G, easyeda2kicad:LED0402-RD_GREEN
- removed P1, P2, P3, P4: PAD, personal_footprint:pad1520oval
- removed U1, U2: 2060-452/998-404, easyeda2kicad:CONN-SMD_2060-452
- added BUZZER1: KLJ-5030, easyeda2kicad:BUZ-SMD_4P-L5.0-W5.0-P3.80-TL, F.Cu at (160.2, 112.5)
- added C2: 2.2uF, Capacitor_SMD:C_0603_1608Metric, F.Cu at (151.9, 106.4)
- added C3: 100nF, Capacitor_SMD:C_0402_1005Metric, F.Cu at (150.6, 105.8)
- added C4: 220uF, easyeda2kicad:CAP-SMD_L3.5-W2.8-FD, F.Cu at (164.9, 105.3)
- added C5: 220uF, easyeda2kicad:CAP-SMD_L3.5-W2.8-FD, F.Cu at (167.9, 114.0)
- added C6: 220uF, easyeda2kicad:CAP-SMD_L3.5-W2.8-FD, F.Cu at (167.9, 105.3)
- added C7: 220uF, easyeda2kicad:CAP-SMD_L3.5-W2.8-FD, F.Cu at (164.9, 109.7)
- added C8: 220uF, easyeda2kicad:CAP-SMD_L3.5-W2.8-FD, F.Cu at (167.9, 109.7)
- added C9: 220uF, easyeda2kicad:CAP-SMD_L3.5-W2.8-FD, F.Cu at (164.9, 114.0)
- added J2: Conn_ARM_SWD_TagConnect_TC2030-NL, Connector:Tag-Connect_TC2030-IDC-NL_2x03_P1.27mm_Vertical, B.Cu at (133.9, 109.1)
- added J3: ~, easyeda2kicad:CONN-TH_XY118-5.0-2P, F.Cu at (179.5, 109.6)
- added J4: ~, easyeda2kicad:CONN-TH_XY118-5.0-2P, F.Cu at (126.7, 109.6)
- added LED1: XL-5050RGBC-WS2812B, easyeda2kicad:LED-SMD_4P-L5.0-W5.0-BL_XL-5050RGBC, F.Cu at (160.1, 107.0)
- added Q3: BSS138LT3G, personal_footprint:SOT96P237X111-3N, F.Cu at (140.6, 105.9)
- added R10: 6.04k, Resistor_SMD:R_0201_0603Metric, F.Cu at (145.2, 104.8)
- added R11: 6.04k, Resistor_SMD:R_0201_0603Metric, F.Cu at (143.9, 107.1)
- added R6: 10k, Resistor_SMD:R_0201_0603Metric, F.Cu at (143.0, 105.0)
- added R7: 10k, Resistor_SMD:R_0201_0603Metric, F.Cu at (150.9, 104.5)
- added R8: 10k, Resistor_SMD:R_0201_0603Metric, F.Cu at (144.1, 105.2)
- added R9: 10k, Resistor_SMD:R_0201_0603Metric, F.Cu at (143.9, 106.3)
- added U3: STM32C011F4Ux, Package_DFN_QFN:ST_UFQFPN-20_3x3mm_P0.5mm, F.Cu at (147.9, 105.8)
- added U4: XC6206P332MR, easyeda2kicad:SOT-23-3_L2.9-W1.6-P1.90-LS2.8-BR, F.Cu at (154.8, 105.7)
- R1, R2, R3: footprint Resistor_SMD:R_0402_1005Metric -> Resistor_SMD:R_0201_0603Metric
- R4: value 150 -> 1k; footprint Resistor_SMD:R_0402_1005Metric -> Resistor_SMD:R_0201_0603Metric
- R5: value 150 -> 6.04k; footprint Resistor_SMD:R_0402_1005Metric -> Resistor_SMD:R_0201_0603Metric
- moved Q2 15.3 mm to (138.8, 108.0), turned to 0 degrees
- moved R5 13.9 mm to (152.3, 104.5), turned to 180 degrees
- moved R1 13.5 mm to (143.1, 108.8)
- moved J1 12.3 mm to (176.0, 112.2), turned to 180 degrees
- moved R2 10.3 mm to (141.7, 108.5), turned to 0 degrees
- moved Q1 10.3 mm to (140.9, 112.4)
- moved R3 6.31 mm to (141.7, 109.2), turned to 0 degrees
- moved R4 4.36 mm to (144.1, 104.4), turned to 0 degrees
- moved SW1 3.86 mm to (150.3, 108.5)
Connections:
- net /TRIGGER_2 renamed Net-(Q1-G)
- J1 pad 2: /TRIGGER -> /IN1
- J1 pad 3: /5V_IN -> /5V0
- Q1 pad 1: /5V_IN -> /FET_5V0
- Q1 pad 2: /5V_IN -> /FET_5V0
- Q1 pad 3: /5V_IN -> /FET_5V0
- Q1 pad 5: /FET_OUT -> /DET_OUT+
- R1 pad 2: /5V_IN -> /FET_5V0
- R3 pad 1: /FET_OUT -> /DET_OUT+
- R4 pad 1: /FET_OUT -> /3V3
- R5 pad 1: /5V_IN -> /IN1
- R5 pad 2: Net-(D2-A) -> /IN1_SENSE
- SW1 pad 1: /DET_OUT+ -> /FET_5V0
- SW1 pad 2: /FET_OUT -> /5V0
Routing:
- net /3V3: track 0.00 -> 64.0 mm, vias 0 -> 3
- net /5V_IN: track 63.2 -> 0.00 mm, vias 10 -> 0
- net /FET_OUT: track 42.6 -> 0.00 mm, vias 8 -> 0
- net /5V0: track 0.00 -> 41.6 mm, vias 0 -> 4
- net /IN2: track 0.00 -> 40.8 mm
- net Net-(BUZZER1--): track 0.90 -> 34.8 mm, vias 0 -> 3
- net /IN1: track 0.00 -> 27.7 mm
- net /SWDIO: track 0.00 -> 24.5 mm, vias 0 -> 1
- net /SWCLK: track 0.00 -> 22.4 mm, vias 0 -> 1
- net /NRST: track 0.00 -> 18.8 mm, vias 0 -> 1
- net /RGB_LED: track 0.00 -> 18.3 mm
- net /FET_5V0: track 0.00 -> 12.5 mm
- net /BUZZER: track 0.00 -> 5.97 mm
- net /IN1_SENSE: track 0.00 -> 3.85 mm
- net GND: track 9.70 -> 13.3 mm, vias 112 -> 12
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- added copper zone on B.Cu, net /5V0
- added copper zone on F.Cu, net /5V0
Other:
- board size 40.3 x 16.2 mm -> 60.9 x 16.1 mm
- board text added: "V2.0"
- board text removed: "DET"
- board text removed: "OUT"
- board text removed: "PWR"
- board text removed: "V1.0"
