File: drone_controller.kicad_sch (KiCad schematic)
At the start: 18 parts, among them J1 Conn_01x03_Pin, P1 PAD, P2 PAD, P3 PAD, P4 PAD, Q1 AGM60P100A, Q2 BSS138LT3G, SW1 SW_SPDT, U1 2060-452/998-404, U2 2060-452/998-404

Commit message: v2.0 release production freeze
Parts:
- removed C1: C_Polarized, easyeda2kicad:CAP-TH_BD8.0-P3.50-D0.6-FD, symbol Device:C_Polarized
- removed D1: LED_R, easyeda2kicad:LED0402-RD, symbol Device:LED
- removed D2: LED_G, easyeda2kicad:LED0402-RD_GREEN, symbol Device:LED
- removed P1, P2, P3, P4: PAD, personal_footprint:pad1520oval, symbol personal_footprint:pad_1
- removed U1, U2: 2060-452/998-404, easyeda2kicad:CONN-SMD_2060-452, symbol easyeda2kicad:2060-452_998-404
- added BUZZER1: KLJ-5030, easyeda2kicad:BUZ-SMD_4P-L5.0-W5.0-P3.80-TL, symbol easyeda2kicad:KLJ-5030
- added C2: 2.2uF, Capacitor_SMD:C_0603_1608Metric, symbol Device:C
- added C3: 100nF, Capacitor_SMD:C_0402_1005Metric, symbol Device:C
- added C4, C5, C6, C7, C8, C9: 220uF, easyeda2kicad:CAP-SMD_L3.5-W2.8-FD, symbol Device:C_Polarized
- added J2: Conn_ARM_SWD_TagConnect_TC2030-NL, Connector:Tag-Connect_TC2030-IDC-NL_2x03_P1.27mm_Vertical, symbol Connector:Conn_ARM_SWD_TagConnect_TC2030-NL
- added J3, J4: ~, easyeda2kicad:CONN-TH_XY118-5.0-2P, symbol personal_footprint:xy118_5.0_2p
- added LED1: XL-5050RGBC-WS2812B, easyeda2kicad:LED-SMD_4P-L5.0-W5.0-BL_XL-5050RGBC, symbol easyeda2kicad:XL-5050RGBC-WS2812B
- added Q3: BSS138LT3G, personal_footprint:SOT96P237X111-3N, symbol personal_footprint:BSS138LT3G
- added R10, R11: 6.04k, Resistor_SMD:R_0201_0603Metric, symbol Device:R
- added R6, R7, R8, R9: 10k, Resistor_SMD:R_0201_0603Metric, symbol Device:R
- added U3: STM32C011F4Ux, Package_DFN_QFN:ST_UFQFPN-20_3x3mm_P0.5mm, symbol MCU_ST_STM32C0:STM32C011F4Ux
- added U4: XC6206P332MR, easyeda2kicad:SOT-23-3_L2.9-W1.6-P1.90-LS2.8-BR, symbol easyeda2kicad:XC6206P332MR
- Q2: LCSC Part (none) -> BSS138LT3G; Manufacturer_Part_Number BSS138LT3G -> (none); Mouser Part Number 863-BSS138LT3G -> (none)
- R1, R2, R3: footprint Resistor_SMD:R_0402_1005Metric -> Resistor_SMD:R_0201_0603Metric; LCSC Part (none) -> C106225
- R4: value 100 -> 1k; footprint Resistor_SMD:R_0402_1005Metric -> Resistor_SMD:R_0201_0603Metric; LCSC Part (none) -> C138165
- R5: value 2k -> 6.04k; footprint Resistor_SMD:R_0402_1005Metric -> Resistor_SMD:R_0201_0603Metric; LCSC Part (none) -> C364363
- SW1: LCSC Part (none) -> D2HW-BL201DL
Connections:
- net DET_OUT+: now also Q1.5 (D), R3.1, J4.1; no longer SW1.1 (B)
- net GND: now also C2.2, C3.2, C4.2, C5.2, C6.2, C7.2, C8.2, C9.2, J2.5 (GND), J4.2, LED1.3 (GND), Q3.2 (S), R6.2, R7.2, R8.2, R9.2, U3.3 (VSS), U4.1 (GND)
- net TRIGGER: now also U3.14 (PA9/PA11); no longer J1.2 (Pin_2)
- net at R4.2: now also BUZZER1.2 (-), Q3.3 (D)
- net IN1_SENSE: now reaches R5.2
- net IN1_SENSE: now also R7.1, U3.6 (PA1)
- net 5V_IN renamed FET_5V0
- net FET_5V0: now also SW1.1 (B), R11.1; no longer J1.3 (Pin_3), R5.1
- removed net FET_OUT: Q1.5 (D), R3.1, R4.1, SW1.2 (A)
- net TRIGGER_2: no longer names the net of Q1.4 (G), Q2.3 (D), R1.1
- new net 3V3: BUZZER1.1 (+), C2.1, C3.1, C4.1, J2.1 (VCC), R4.1, U3.2 (VDD), U4.3 (Vout)
- new net 5V0: C5.1, C6.1, C7.1, C8.1, C9.1, J1.3 (Pin_3), J3.2, LED1.1 (VDD), SW1.2 (A), U4.2 (Vin)
- new net BUZZER: Q3.1 (G), R6.1, U3.13 (PA8)
- new net FET_5V0_SENSE: R11.2, R9.1, U3.15 (PA10/PA12)
- new net IN1: J1.2 (Pin_2), R5.1
- new net IN2: J3.1, R10.1
- new net IN2_SENSE: R10.2, R8.1, U3.12 (PA7)
- new net NRST: J2.3 (~{RESET}), U3.4 (PF2)
- new net RGB_LED: LED1.4 (DIN), U3.1 (PC15)
- new net SWCLK: J2.4 (SWCLK), U3.17 (PA14)
- new net SWDIO: J2.2 (SWDIO), U3.16 (PA13)
- no-connect marks 0 -> 12
Other:
- note added: "5V0"
- note removed: "5V_IN"
- moved on the sheet: J1, Q1, Q2, SW1
